Commit message: Rename joints to *_joint and fix shoulder typo
Fix hand_link <collsion> tag and add its SRDF collision pairs

File: arm_description/urdf/arm.xacro (robot description, xacro)
@@ -99,13 +99,13 @@
             <material name="grey" />
         </visual>
-        <collsion>
+        <collision>
             <geometry>
                 <box size="0.1 0.1 0.02" />
             </geometry>
             <origin xyz="0 0 0.01" rpy="0 0 0" />
-        </collsion>
+        </collision>
     </link>
     <link name="tool_link" />
-    <joint name="base_shoulder_link" type="revolute">
+    <joint name="base_shoulder_joint" type="revolute">
         <parent link="base_link" />
         <child link="shoulder_link" />
@@ -114,5 +114,5 @@
         <limit effort="1000.0" velocity="1.0" lower="-3.14" upper="3.14" />
     </joint>
-    <joint name="shoudler_arm_link" type="revolute">
+    <joint name="shoulder_arm_joint" type="revolute">
         <parent link="shoulder_link" />
         <child link="arm_link" />
@@ -121,5 +121,5 @@
         <limit effort="1000.0" velocity="1.0" lower="0" upper="2.5" />
     </joint>
-    <joint name="arm_elbow_link" type="revolute">
+    <joint name="arm_elbow_joint" type="revolute">
         <parent link="arm_link" />
         <child link="elbow_link" />
@@ -128,5 +128,5 @@
         <limit effort="1000.0" velocity="1.0" lower="0" upper="2.5" />
     </joint>
-    <joint name="elbow_forearm_link" type="revolute">
+    <joint name="elbow_forearm_joint" type="revolute">
         <parent link="elbow_link" />
         <child link="forearm_link" />
@@ -135,5 +135,5 @@
         <limit effort="1000.0" velocity="1.0" lower="-3.14" upper="3.14" />
     </joint>
-    <joint name="forearm_wrist_link" type="revolute">
+    <joint name="forearm_wrist_joint" type="revolute">
         <parent link="forearm_link" />
         <child link="wrist_link" />
@@ -142,5 +142,5 @@
         <limit effort="1000.0" velocity="1.0" lower="-1.57" upper="1.57" />
     </joint>
-    <joint name="wrist_hand_link" type="continuous">
+    <joint name="wrist_hand_joint" type="continuous">
         <parent link="wrist_link" />
         <child link="hand_link" />

File: arm_description/urdf/robot_arm.ros2_control.xacro (robot description, xacro)
@@ -6,5 +6,5 @@
           <plugin>mock_components/GenericSystem</plugin>
       </hardware>
-      <joint name="base_shoulder_link">
+      <joint name="base_shoulder_joint">
           <command_interface name="position"/>
           <state_interface name="position">
@@ -12,5 +12,5 @@
           </state_interface>
       </joint>
-      <joint name="shoudler_arm_link">
+      <joint name="shoulder_arm_joint">
           <command_interface name="position"/>
           <state_interface name="position">
@@ -18,5 +18,5 @@
           </state_interface>
       </joint>
-      <joint name="arm_elbow_link">
+      <joint name="arm_elbow_joint">
           <command_interface name="position"/>
           <state_interface name="position">
@@ -24,5 +24,5 @@
           </state_interface>
       </joint>
-      <joint name="elbow_forearm_link">
+      <joint name="elbow_forearm_joint">
           <command_interface name="position"/>
           <state_interface name="position">
@@ -30,5 +30,5 @@
           </state_interface>
       </joint>
-      <joint name="forearm_wrist_link">
+      <joint name="forearm_wrist_joint">
           <command_interface name="position"/>
           <state_interface name="position">
@@ -36,5 +36,5 @@
           </state_interface>
       </joint>
-      <joint name="wrist_hand_link">
+      <joint name="wrist_hand_joint">
           <command_interface name="position"/>
           <state_interface name="position">

File: arm_moveit_config/config/robot_arm.ros2_control.xacro (robot description, xacro)
@@ -8,38 +8,38 @@
                 <plugin>mock_components/GenericSystem</plugin>
             </hardware>
-            <joint name="base_shoulder_link">
+            <joint name="base_shoulder_joint">
                 <command_interface name="position"/>
                 <state_interface name="position">
-                  <param name="initial_value">${initial_positions['base_shoulder_link']}</param>
+                  <param name="initial_value">${initial_positions['base_shoulder_joint']}</param>
                 </state_interface>
             </joint>
-            <joint name="shoudler_arm_link">
+            <joint name="shoulder_arm_joint">
                 <command_interface name="position"/>
                 <state_interface name="position">
-                  <param name="initial_value">${initial_positions['shoudler_arm_link']}</param>
+                  <param name="initial_value">${initial_positions['shoulder_arm_joint']}</param>
                 </state_interface>
             </joint>
-            <joint name="arm_elbow_link">
+            <joint name="arm_elbow_joint">
                 <command_interface name="position"/>
                 <state_interface name="position">
-                  <param name="initial_value">${initial_positions['arm_elbow_link']}</param>
+                  <param name="initial_value">${initial_positions['arm_elbow_joint']}</param>
                 </state_interface>
             </joint>
-            <joint name="elbow_forearm_link">
+            <joint name="elbow_forearm_joint">
                 <command_interface name="position"/>
                 <state_interface name="position">
-                  <param name="initial_value">${initial_positions['elbow_forearm_link']}</param>
+                  <param name="initial_value">${initial_positions['elbow_forearm_joint']}</param>
                 </state_interface>
             </joint>
-            <joint name="forearm_wrist_link">
+            <joint name="forearm_wrist_joint">
                 <command_interface name="position"/>
                 <state_interface name="position">
-                  <param name="initial_value">${initial_positions['forearm_wrist_link']}</param>
+                  <param name="initial_value">${initial_positions['forearm_wrist_joint']}</param>
                 </state_interface>
             </joint>
-            <joint name="wrist_hand_link">
+            <joint name="wrist_hand_joint">
                 <command_interface name="position"/>
                 <state_interface name="position">
-                  <param name="initial_value">${initial_positions['wrist_hand_link']}</param>
+                  <param name="initial_value">${initial_positions['wrist_hand_joint']}</param>
                 </state_interface>
             </joint>

Commit message: Add mass and inertia to all arm and gripper links
Box and cylinder inertia macros in common_properties.xacro

File: arm_description/urdf/arm.xacro (robot description, xacro)
@@ -15,4 +15,5 @@
             <origin xyz="0 0 0.05" rpy="0 0 0" />
         </collision>
+        <xacro:box_inertia m="5.0" x="0.4" y="0.4" z="0.1" xyz="0 0 0.05" />
     </link>
     <link name="shoulder_link">
@@ -30,4 +31,5 @@
             <origin xyz="0 0 0.25" rpy="0 0 0" />
         </collision>
+        <xacro:cylinder_inertia m="2.0" r="0.1" l="0.5" xyz="0 0 0.25" />
     </link>
     <link name="arm_link">
@@ -45,4 +47,5 @@
             <origin xyz="0 0 0.3" rpy="0 0 0" />
         </collision>
+        <xacro:cylinder_inertia m="1.5" r="0.05" l="0.6" xyz="0 0 0.3" />
     </link>
     <link name="elbow_link">
@@ -60,4 +63,5 @@
             <origin xyz="0 0 0.05" rpy="0 0 0" />
         </collision>
+        <xacro:cylinder_inertia m="0.3" r="0.05" l="0.1" xyz="0 0 0.05" />
     </link>
     <link name="forearm_link">
@@ -75,4 +79,5 @@
             <origin xyz="0 0 0.25" rpy="0 0 0" />
         </collision>
+        <xacro:cylinder_inertia m="1.0" r="0.05" l="0.5" xyz="0 0 0.25" />
     </link>
     <link name="wrist_link">
@@ -90,4 +95,5 @@
             <origin xyz="0 0 0.025" rpy="0 0 0" />
         </collision>
+        <xacro:box_inertia m="0.3" x="0.1" y="0.1" z="0.05" xyz="0 0 0.025" />
     </link>
     <link name="hand_link">
@@ -105,4 +111,5 @@
             <origin xyz="0 0 0.01" rpy="0 0 0" />
         </collision>
+        <xacro:box_inertia m="0.2" x="0.1" y="0.1" z="0.02" xyz="0 0 0.01" />
     </link>
     <link name="tool_link" />

File: arm_description/urdf/common_properties.xacro (robot description, xacro)
@@ -13,3 +13,22 @@
         <color rgba="0 0.6 0 1" />
     </material>
+    <!-- Solid box / cylinder (axis along z) inertia, centred at xyz -->
+    <xacro:macro name="box_inertia" params="m x y z xyz">
+        <inertial>
+            <origin xyz="${xyz}" rpy="0 0 0" />
+            <mass value="${m}" />
+            <inertia ixx="${m*(y*y+z*z)/12}" ixy="0" ixz="0"
+                     iyy="${m*(x*x+z*z)/12}" iyz="0"
+                     izz="${m*(x*x+y*y)/12}" />
+        </inertial>
+    </xacro:macro>
+    <xacro:macro name="cylinder_inertia" params="m r l xyz">
+        <inertial>
+            <origin xyz="${xyz}" rpy="0 0 0" />
+            <mass value="${m}" />
+            <inertia ixx="${m*(3*r*r+l*l)/12}" ixy="0" ixz="0"
+                     iyy="${m*(3*r*r+l*l)/12}" iyz="0"
+                     izz="${m*r*r/2}" />
+        </inertial>
+    </xacro:macro>
 </robot>

File: arm_description/urdf/gripper.xacro (robot description, xacro)
@@ -15,4 +15,5 @@
             <origin xyz="0 0 0.01" rpy="0 0 0" />
         </collision>
+        <xacro:box_inertia m="0.2" x="0.2" y="0.06" z="0.02" xyz="0 0 0.01" />
     </link>
     <link name="gripper_left_finger_link">
@@ -30,4 +31,5 @@
             <origin xyz="0 0 0.04" rpy="0 0 0" />
         </collision>
+        <xacro:box_inertia m="0.05" x="0.02" y="0.06" z="0.08" xyz="0 0 0.04" />
     </link>
     <link name="gripper_right_finger_link">
@@ -45,4 +47,5 @@
             <origin xyz="0 0 0.04" rpy="0 0 0" />
         </collision>
+        <xacro:box_inertia m="0.05" x="0.02" y="0.06" z="0.08" xyz="0 0 0.04" />
     </link>
     <joint name="gripper_left_finger_joint" type="prismatic">
