Commit message: Add sim xacro arg to switch between mock and Gazebo hardware
Sim mode fixes base to world, loads gz_ros2_control; lower finger effort limit

File: arm_description/urdf/gripper.xacro (robot description, xacro)
@@ -54,5 +54,5 @@
         <origin xyz="-0.07 0 0.02" rpy="0 0 0" />
         <axis xyz="1 0 0" />
-        <limit effort="1000.0" velocity="1.0" lower="0.0" upper="0.06" />
+        <limit effort="50.0" velocity="1.0" lower="0.0" upper="0.06" />
     </joint>
     <joint name="gripper_right_finger_joint" type="prismatic">
@@ -62,5 +62,5 @@
         <axis xyz="1 0 0" />
         <mimic joint="gripper_left_finger_joint" multiplier="-1.0" />
-        <limit effort="1000.0" velocity="1.0" lower="-0.06" upper="0.0" />
+        <limit effort="50.0" velocity="1.0" lower="-0.06" upper="0.0" />
     </joint>
 </robot>

File: arm_description/urdf/robot_arm.ros2_control.xacro (robot description, xacro)
@@ -3,6 +3,10 @@
   <ros2_control name="Arm" type="system">
       <hardware>
-          <!-- By default, set up controllers for simulation. This won't work on real hardware -->
-          <plugin>mock_components/GenericSystem</plugin>
+          <xacro:if value="$(arg sim)">
+              <plugin>gz_ros2_control/GazeboSimSystem</plugin>
+          </xacro:if>
+          <xacro:unless value="$(arg sim)">
+              <plugin>mock_components/GenericSystem</plugin>
+          </xacro:unless>
       </hardware>
       <joint name="base_shoulder_joint">
@@ -48,4 +52,10 @@
           </state_interface>
       </joint>
+      <xacro:if value="$(arg sim)">
+          <!-- Mimics the left finger; Gazebo moves it, ros2_control only reads it -->
+          <joint name="gripper_right_finger_joint">
+              <state_interface name="position"/>
+          </joint>
+      </xacro:if>
   </ros2_control>
 </robot>

File: arm_description/urdf/robot_arm.urdf.xacro (robot description, xacro)
@@ -1,4 +1,6 @@
 <?xml version="1.0"?>
 <robot name="robot_arm" xmlns:xacro="http://www.ros.org/wiki/xacro">
+    <!-- sim:=true runs on Gazebo (gz_ros2_control); default is mock hardware -->
+    <xacro:arg name="sim" default="false" />
     <xacro:include filename="common_properties.xacro" />
     <xacro:include filename="arm.xacro" />
@@ -10,3 +12,16 @@
         <origin xyz="0 0 0" rpy="0 0 0" />
     </joint>
+    <xacro:if value="$(arg sim)">
+        <!-- Bolt the base to the ground. Sim only: MoveIt adds its own world joint from the SRDF -->
+        <link name="world" />
+        <joint name="world_base_joint" type="fixed">
+            <parent link="world" />
+            <child link="base_link" />
+        </joint>
+        <gazebo>
+            <plugin filename="gz_ros2_control-system" name="gz_ros2_control::GazeboSimROS2ControlPlugin">
+                <parameters>$(find arm_bringup)/config/ros2_controllers.yaml</parameters>
+            </plugin>
+        </gazebo>
+    </xacro:if>
 </robot>

Commit message: Drive gripper fingers by force as two separate joints
Drop the mimic so both fingers close together in Gazebo; they squeeze with a capped effort and higher friction.

File: arm_description/urdf/gripper.xacro (robot description, xacro)
@@ -1,4 +1,6 @@
 <?xml version="1.0"?>
 <robot xmlns:xacro="http://www.ros.org/wiki/xacro">
+    <!-- Max squeeze per finger in Gazebo (N). Effort commands are capped here -->
+    <xacro:property name="FINGER_FORCE" value="15.0" />
     <link name="gripper_base_link">
         <visual>
@@ -31,5 +33,7 @@
             <origin xyz="0 0 0.04" rpy="0 0 0" />
         </collision>
-        <xacro:box_inertia m="0.05" x="0.02" y="0.06" z="0.08" xyz="0 0 0.04" />
+        <!-- Two Gazebo workarounds so both fingers move together. Fingers not lighter than this, and
+             joint ranges starting 1 cm below open (0), since a finger resting on its limit can stall -->
+        <xacro:box_inertia m="0.2" x="0.02" y="0.06" z="0.08" xyz="0 0 0.04" />
     </link>
     <link name="gripper_right_finger_link">
@@ -47,5 +51,5 @@
             <origin xyz="0 0 0.04" rpy="0 0 0" />
         </collision>
-        <xacro:box_inertia m="0.05" x="0.02" y="0.06" z="0.08" xyz="0 0 0.04" />
+        <xacro:box_inertia m="0.2" x="0.02" y="0.06" z="0.08" xyz="0 0 0.04" />
     </link>
     <joint name="gripper_left_finger_joint" type="prismatic">
@@ -54,5 +58,5 @@
         <origin xyz="-0.07 0 0.02" rpy="0 0 0" />
         <axis xyz="1 0 0" />
-        <limit effort="50.0" velocity="1.0" lower="0.0" upper="0.06" />
+        <limit effort="${FINGER_FORCE}" velocity="1.0" lower="-0.01" upper="0.06" />
     </joint>
     <joint name="gripper_right_finger_joint" type="prismatic">
@@ -60,7 +64,7 @@
         <child link="gripper_right_finger_link" />
         <origin xyz="0.07 0 0.02" rpy="0 0 0" />
-        <axis xyz="1 0 0" />
-        <mimic joint="gripper_left_finger_joint" multiplier="-1.0" />
-        <limit effort="50.0" velocity="1.0" lower="-0.06" upper="0.0" />
+        <!-- Mirrored axis so both fingers close with the same positive value -->
+        <axis xyz="-1 0 0" />
+        <limit effort="${FINGER_FORCE}" velocity="1.0" lower="-0.01" upper="0.06" />
     </joint>
 </robot>

File: arm_description/urdf/robot_arm.ros2_control.xacro (robot description, xacro)
@@ -46,16 +46,23 @@
           </state_interface>
       </joint>
-      <joint name="gripper_left_finger_joint">
-          <command_interface name="position"/>
-          <state_interface name="position">
-            <param name="initial_value">0.0</param>
-          </state_interface>
-      </joint>
-      <xacro:if value="$(arg sim)">
-          <!-- Mimics the left finger; Gazebo moves it, ros2_control only reads it -->
-          <joint name="gripper_right_finger_joint">
-              <state_interface name="position"/>
+      <!-- Fingers: position on mock hardware; in Gazebo they push with a force (effort) so the
+           grip is a set squeeze instead of whatever a stalled position servo produces -->
+      <xacro:macro name="finger" params="name">
+          <joint name="${name}">
+              <xacro:if value="$(arg sim)">
+                  <command_interface name="effort"/>
+                  <state_interface name="position"/>
+                  <state_interface name="velocity"/>
+              </xacro:if>
+              <xacro:unless value="$(arg sim)">
+                  <command_interface name="position"/>
+                  <state_interface name="position">
+                    <param name="initial_value">0.0</param>
+                  </state_interface>
+              </xacro:unless>
           </joint>
-      </xacro:if>
+      </xacro:macro>
+      <xacro:finger name="gripper_left_finger_joint"/>
+      <xacro:finger name="gripper_right_finger_joint"/>
   </ros2_control>
 </robot>

File: arm_description/urdf/robot_arm.urdf.xacro (robot description, xacro)
@@ -23,14 +23,14 @@
         <!-- Grippy fingers so the box doesn't slip out -->
         <gazebo reference="gripper_left_finger_link">
-            <mu1>1.5</mu1>
-            <mu2>1.5</mu2>
+            <mu1>2.0</mu1>
+            <mu2>2.0</mu2>
         </gazebo>
         <gazebo reference="gripper_right_finger_link">
-            <mu1>1.5</mu1>
-            <mu2>1.5</mu2>
+            <mu1>2.0</mu1>
+            <mu2>2.0</mu2>
         </gazebo>
         <gazebo>
             <plugin filename="gz_ros2_control-system" name="gz_ros2_control::GazeboSimROS2ControlPlugin">
-                <parameters>$(find arm_bringup)/config/ros2_controllers.yaml</parameters>
+                <parameters>$(find arm_bringup)/config/ros2_controllers_gz.yaml</parameters>
             </plugin>
         </gazebo>

File: arm_moveit_config/config/robot_arm.ros2_control.xacro (robot description, xacro)
@@ -50,4 +50,10 @@
                 </state_interface>
             </joint>
+            <joint name="gripper_right_finger_joint">
+                <command_interface name="position"/>
+                <state_interface name="position">
+                  <param name="initial_value">${initial_positions['gripper_right_finger_joint']}</param>
+                </state_interface>
+            </joint>
         </ros2_control>
     </xacro:macro>
